File: ModelRocketAvionicsPCB/Sensors.sch (KiCad schematic (older format))
At the start: 17 parts

Commit message: Annotated components and added 'Digi-Key Part Numbers' for most of the non-passives
Parts:
- U3: renamed from U?; Digi-Key Part Number (none) -> 497-10134-ND
- U4: renamed from U?; Digi-Key Part Number (none) -> 497-13931-1-ND
- U5: renamed from U?; Digi-Key Part Number (none) -> MPL3115A2-ND
- gave numbers to parts that had none: 14
Changed lines of the file:
@@
 $EndDescr
 $Comp
-L MPL3115A2 U?
+L MPL3115A2 U5
 U 1 1 5AE7793E
 P 5800 1600
-F 0 "U?" H 5800 1750 60  0000 C CNN
+F 0 "U5" H 5800 1750 60  0000 C CNN
 F 1 "MPL3115A2" H 5800 2000 60  0000 C CNN
 F 2 "" H 5800 1600 60  0001 C CNN
 F 3 "" H 5800 1600 60  0001 C CNN
+F 4 "MPL3115A2-ND" H 5800 1600 60  0001 C CNN "Digi-Key Part Number"
 	1    5800 1600
 	1    0    0    -1
 $EndComp
 $Comp
-L LIS331 U?
+L LIS331 U3
 U 1 1 5AE779FB
 P 5650 3450
-F 0 "U?" H 5800 3600 60  0000 C CNN
+F 0 "U3" H 5800 3600 60  0000 C CNN
 F 1 "LIS331" H 5800 3700 60  0000 C CNN
 F 2 "" H 5650 3450 60  0001 C CNN
 F 3 "" H 5650 3450 60  0001 C CNN
+F 4 "497-10134-ND" H 5650 3450 60  0001 C CNN "Digi-Key Part Number"
 	1    5650 3450
 	1    0    0    -1
 $EndComp
 $Comp
-L L3GD20HTR U?
+L L3GD20HTR U4
 U 1 1 5AE77A26
 P 5700 5500
-F 0 "U?" H 5950 5350 60  0000 C CNN
+F 0 "U4" H 5950 5350 60  0000 C CNN
 F 1 "L3GD20HTR" H 5850 5450 60  0000 C CNN
 F 2 "" H 5700 5500 60  0001 C CNN
 F 3 "" H 5700 5500 60  0001 C CNN
+F 4 "497-13931-1-ND" H 5700 5500 60  0001 C CNN "Digi-Key Part Number"
 	1    5700 5500
 	1    0    0    -1
@@
 NoConn ~ 5250 3200
 $Comp
-L +3V3 #PWR09
+L +3V3 #PWR24
 U 1 1 5AE77CF8
 P 3600 3100
-F 0 "#PWR09" H 3600 2950 50  0001 C CNN
+F 0 "#PWR24" H 3600 2950 50  0001 C CNN
 F 1 "+3V3" H 3600 3240 50  0000 C CNN
 F 2 "" H 3600 3100 50  0000 C CNN
@@
 $EndComp
 $Comp
-L CP1 C?
+L CP1 C21
 U 1 1 5AE77D1E
 P 3400 3500
-F 0 "C?" H 3425 3600 50  0000 L CNN
+F 0 "C21" H 3425 3600 50  0000 L CNN
 F 1 "10uF" H 3425 3400 50  0000 L CNN
 F 2 "" H 3400 3500 50  0000 C CNN
@@
 $EndComp
 $Comp
-L C C?
+L C C24
 U 1 1 5AE77DC3
 P 3800 3500
-F 0 "C?" H 3825 3600 50  0000 L CNN
+F 0 "C24" H 3825 3600 50  0000 L CNN
 F 1 "0.1uF" H 3825 3400 50  0000 L CNN
 F 2 "" H 3838 3350 50  0000 C CNN
@@
 $EndComp
 $Comp
-L GND #PWR010
+L GND #PWR25
 U 1 1 5AE77F37
 P 3600 3900
-F 0 "#PWR010" H 3600 3650 50  0001 C CNN
+F 0 "#PWR25" H 3600 3650 50  0001 C CNN
 F 1 "GND" H 3600 3750 50  0000 C CNN
 F 2 "" H 3600 3900 50  0000 C CNN
@@
 $EndComp
 $Comp
-L GND #PWR011
+L GND #PWR35
 U 1 1 5AE77FFB
 P 7100 3950
-F 0 "#PWR011" H 7100 3700 50  0001 C CNN
+F 0 "#PWR35" H 7100 3700 50  0001 C CNN
 F 1 "GND" H 7100 3800 50  0000 C CNN
 F 2 "" H 7100 3950 50  0000 C CNN
@@
 $EndComp
 $Comp
-L +3V3 #PWR012
+L +3V3 #PWR31
 U 1 1 5AE7810D
 P 6500 3000
-F 0 "#PWR012" H 6500 2850 50  0001 C CNN
+F 0 "#PWR31" H 6500 2850 50  0001 C CNN
 F 1 "+3V3" H 6500 3140 50  0000 C CNN
 F 2 "" H 6500 3000 50  0000 C CNN
@@
 $EndComp
 $Comp
-L +3V3 #PWR013
+L +3V3 #PWR30
 U 1 1 5AE7815D
 P 5150 3000
-F 0 "#PWR013" H 5150 2850 50  0001 C CNN
+F 0 "#PWR30" H 5150 2850 50  0001 C CNN
 F 1 "+3V3" H 5150 3140 50  0000 C CNN
 F 2 "" H 5150 3000 50  0000 C CNN
@@
 $EndComp
 $Comp
-L GND #PWR014
+L GND #PWR26
 U 1 1 5AE78194
 P 4600 3950
-F 0 "#PWR014" H 4600 3700 50  0001 C CNN
+F 0 "#PWR26" H 4600 3700 50  0001 C CNN
 F 1 "GND" H 4600 3800 50  0000 C CNN
 F 2 "" H 4600 3950 50  0000 C CNN
@@
 ACC_LSB
 $Comp
-L Jumper_NC_Small JP?
+L Jumper_NC_Small JP2
 U 1 1 5AE7870B
 P 8550 3600
-F 0 "JP?" H 8550 3680 50  0000 C CNN
+F 0 "JP2" H 8550 3680 50  0000 C CNN
 F 1 "Jumper_NC_Small" H 8560 3540 50  0001 C CNN
 F 2 "" H 8550 3600 50  0000 C CNN
@@
 $EndComp
 $Comp
-L Jumper_NO_Small JP?
+L Jumper_NO_Small JP1
 U 1 1 5AE78786
 P 8550 3300
-F 0 "JP?" H 8550 3380 50  0000 C CNN
+F 0 "JP1" H 8550 3380 50  0000 C CNN
 F 1 "Jumper_NO_Small" H 8560 3240 50  0001 C CNN
 F 2 "" H 8550 3300 50  0000 C CNN
@@
 $EndComp
 $Comp
-L +3V3 #PWR015
+L +3V3 #PWR36
 U 1 1 5AE7881C
 P 8750 3200
-F 0 "#PWR015" H 8750 3050 50  0001 C CNN
+F 0 "#PWR36" H 8750 3050 50  0001 C CNN
 F 1 "+3V3" H 8750 3340 50  0000 C CNN
 F 2 "" H 8750 3200 50  0000 C CNN
@@
 $EndComp
 $Comp
-L GND #PWR016
+L GND #PWR37
 U 1 1 5AE7883E
 P 8750 3700
-F 0 "#PWR016" H 8750 3450 50  0001 C CNN
+F 0 "#PWR37" H 8750 3450 50  0001 C CNN
 F 1 "GND" H 8750 3550 50  0000 C CNN
 F 2 "" H 8750 3700 50  0000 C CNN
@@
 ACC_CS
 $Comp
-L +3V3 #PWR017
+L +3V3 #PWR40
 U 1 1 5AE78BF2
 P 10200 3350
-F 0 "#PWR017" H 10200 3200 50  0001 C CNN
+F 0 "#PWR40" H 10200 3200 50  0001 C CNN
 F 1 "+3V3" H 10200 3490 50  0000 C CNN
 F 2 "" H 10200 3350 50  0000 C CNN
@@
 I2C_SDA
 $Comp
-L GND #PWR018
+L GND #PWR29
 U 1 1 5AE7A26D
 P 5150 1900
-F 0 "#PWR018" H 5150 1650 50  0001 C CNN
+F 0 "#PWR29" H 5150 1650 50  0001 C CNN
 F 1 "GND" H 5150 1750 50  0000 C CNN
 F 2 "" H 5150 1900 50  0000 C CNN
@@
 $EndComp
 $Comp
-L +3V3 #PWR019
+L +3V3 #PWR27
 U 1 1 5AE7A2CF
 P 5100 1250
-F 0 "#PWR019" H 5100 1100 50  0001 C CNN
+F 0 "#PWR27" H 5100 1100 50  0001 C CNN
 F 1 "+3V3" H 5100 1390 50  0000 C CNN
 F 2 "" H 5100 1250 50  0000 C CNN
@@
 $EndComp
 $Comp
-L C C?
+L C C27
 U 1 1 5AE7A368
 P 4800 1650
-F 0 "C?" H 4825 1750 50  0000 L CNN
+F 0 "C27" H 4825 1750 50  0000 L CNN
 F 1 "0.1uF" H 4825 1550 50  0000 L CNN
 F 2 "" H 4838 1500 50  0000 C CNN
@@
 Connection ~ 5150 1850
 $Comp
-L +3V3 #PWR020
+L +3V3 #PWR20
 U 1 1 5AE7AAE0
 P 3450 1100
-F 0 "#PWR020" H 3450 950 50  0001 C CNN
+F 0 "#PWR20" H 3450 950 50  0001 C CNN
 F 1 "+3V3" H 3450 1240 50  0000 C CNN
 F 2 "" H 3450 1100 50  0000 C CNN
@@
 $EndComp
 $Comp
-L CP1 C?
+L CP1 C19
 U 1 1 5AE7AAE6
 P 3050 1500
-F 0 "C?" H 3075 1600 50  0000 L CNN
+F 0 "C19" H 3075 1600 50  0000 L CNN
 F 1 "10uF" H 3075 1400 50  0000 L CNN
 F 2 "" H 3050 1500 50  0000 C CNN
@@
 $EndComp
 $Comp
-L C C?
+L C C22
 U 1 1 5AE7AAEC
 P 3450 1500
-F 0 "C?" H 3475 1600 50  0000 L CNN
+F 0 "C22" H 3475 1600 50  0000 L CNN
 F 1 "0.1uF" H 3475 1400 50  0000 L CNN
 F 2 "" H 3488 1350 50  0000 C CNN
@@
 $EndComp
 $Comp
-L GND #PWR021
+L GND #PWR21
 U 1 1 5AE7AAF2
 P 3450 1900
-F 0 "#PWR021" H 3450 1650 50  0001 C CNN
+F 0 "#PWR21" H 3450 1650 50  0001 C CNN
 F 1 "GND" H 3450 1750 50  0000 C CNN
 F 2 "" H 3450 1900 50  0000 C CNN
@@
 $EndComp
 $Comp
-L C C?
+L C C25
 U 1 1 5AE7AB7A
 P 3850 1500
-F 0 "C?" H 3875 1600 50  0000 L CNN
+F 0 "C25" H 3875 1600 50  0000 L CNN
 F 1 "1uF" H 3875 1400 50  0000 L CNN
 F 2 "" H 3888 1350 50  0000 C CNN
@@
 	5150 5250 5200 5250
 $Comp
-L +3V3 #PWR022
+L +3V3 #PWR28
 U 1 1 5AE7C572
 P 5100 5050
-F 0 "#PWR022" H 5100 4900 50  0001 C CNN
+F 0 "#PWR28" H 5100 4900 50  0001 C CNN
 F 1 "+3V3" H 5100 5190 50  0000 C CNN
 F 2 "" H 5100 5050 50  0000 C CNN
@@
 	5100 5150 5200 5150
 $Comp
-L +3V3 #PWR023
+L +3V3 #PWR32
 U 1 1 5AE7C69B
 P 6600 5050
-F 0 "#PWR023" H 6600 4900 50  0001 C CNN
+F 0 "#PWR32" H 6600 4900 50  0001 C CNN
 F 1 "+3V3" H 6600 5190 50  0000 C CNN
 F 2 "" H 6600 5050 50  0000 C CNN
@@
 Connection ~ 6600 5150
 $Comp
-L GND #PWR024
+L GND #PWR33
 U 1 1 5AE7C886
 P 6600 5950
-F 0 "#PWR024" H 6600 5700 50  0001 C CNN
+F 0 "#PWR33" H 6600 5700 50  0001 C CNN
 F 1 "GND" H 6600 5800 50  0000 C CNN
 F 2 "" H 6600 5950 50  0000 C CNN
@@
 	6500 5450 6600 5450
 $Comp
-L C C?
+L C C28
 U 1 1 5AE7CBFF
 P 6850 5550
-F 0 "C?" H 6875 5650 50  0000 L CNN
+F 0 "C28" H 6875 5650 50  0000 L CNN
 F 1 "10nF(25V)" H 6875 5450 50  0000 L CNN
 F 2 "" H 6888 5400 50  0000 C CNN
@@
 	6850 5350 6500 5350
 $Comp
-L GND #PWR025
+L GND #PWR34
 U 1 1 5AE7CD24
 P 6850 5750
-F 0 "#PWR025" H 6850 5500 50  0001 C CNN
+F 0 "#PWR34" H 6850 5500 50  0001 C CNN
 F 1 "GND" H 6850 5600 50  0000 C CNN
 F 2 "" H 6850 5750 50  0000 C CNN
@@
 Connection ~ 6600 5850
 $Comp
-L +3V3 #PWR026
+L +3V3 #PWR22
 U 1 1 5AE7D7A9
 P 3450 5100
-F 0 "#PWR026" H 3450 4950 50  0001 C CNN
+F 0 "#PWR22" H 3450 4950 50  0001 C CNN
 F 1 "+3V3" H 3450 5240 50  0000 C CNN
 F 2 "" H 3450 5100 50  0000 C CNN
@@
 $EndComp
 $Comp
-L C C?
+L C C23
 U 1 1 5AE7D7B5
 P 3450 5500
-F 0 "C?" H 3475 5600 50  0000 L CNN
+F 0 "C23" H 3475 5600 50  0000 L CNN
 F 1 ".1uF" H 3475 5400 50  0000 L CNN
 F 2 "" H 3488 5350 50  0000 C CNN
@@
 $EndComp
 $Comp
-L GND #PWR027
+L GND #PWR23
 U 1 1 5AE7D7BB
 P 3450 5900
-F 0 "#PWR027" H 3450 5650 50  0001 C CNN
+F 0 "#PWR23" H 3450 5650 50  0001 C CNN
 F 1 "GND" H 3450 5750 50  0000 C CNN
 F 2 "" H 3450 5900 50  0000 C CNN
@@
 $EndComp
 $Comp
-L C C?
+L C C26
 U 1 1 5AE7D7C1
 P 3850 5500
-F 0 "C?" H 3875 5600 50  0000 L CNN
+F 0 "C26" H 3875 5600 50  0000 L CNN
 F 1 ".1uF" H 3875 5400 50  0000 L CNN
 F 2 "" H 3888 5350 50  0000 C CNN
@@
 	3850 5250 3850 5350
 $Comp
-L C C?
+L C C20
 U 1 1 5AE7D9AB
 P 3050 5500
-F 0 "C?" H 3075 5600 50  0000 L CNN
+F 0 "C20" H 3075 5600 50  0000 L CNN
 F 1 "10uF" H 3075 5400 50  0000 L CNN
 F 2 "" H 3088 5350 50  0000 C CNN
@@
 GYR_CS
 $Comp
-L +3V3 #PWR028
+L +3V3 #PWR41
 U 1 1 5AE7E065
 P 10200 5350
-F 0 "#PWR028" H 10200 5200 50  0001 C CNN
+F 0 "#PWR41" H 10200 5200 50  0001 C CNN
 F 1 "+3V3" H 10200 5490 50  0000 C CNN
 F 2 "" H 10200 5350 50  0000 C CNN
@@
 GYR_LSB
 $Comp
-L Jumper_NC_Small JP?
+L Jumper_NC_Small JP4
 U 1 1 5AE7E366
 P 8550 5600
-F 0 "JP?" H 8550 5680 50  0000 C CNN
+F 0 "JP4" H 8550 5680 50  0000 C CNN
 F 1 "Jumper_NC_Small" H 8560 5540 50  0001 C CNN
 F 2 "" H 8550 5600 50  0000 C CNN
@@
 $EndComp
 $Comp
-L Jumper_NO_Small JP?
+L Jumper_NO_Small JP3
 U 1 1 5AE7E36C
 P 8550 5300
-F 0 "JP?" H 8550 5380 50  0000 C CNN
+F 0 "JP3" H 8550 5380 50  0000 C CNN
 F 1 "Jumper_NO_Small" H 8560 5240 50  0001 C CNN
 F 2 "" H 8550 5300 50  0000 C CNN
@@
 $EndComp
 $Comp
-L +3V3 #PWR029
+L +3V3 #PWR38
 U 1 1 5AE7E372
 P 8750 5200
-F 0 "#PWR029" H 8750 5050 50  0001 C CNN
+F 0 "#PWR38" H 8750 5050 50  0001 C CNN
 F 1 "+3V3" H 8750 5340 50  0000 C CNN
 F 2 "" H 8750 5200 50  0000 C CNN
@@
 $EndComp
 $Comp
-L GND #PWR030
+L GND #PWR39
 U 1 1 5AE7E378
 P 8750 5700
-F 0 "#PWR030" H 8750 5450 50  0001 C CNN
+F 0 "#PWR39" H 8750 5450 50  0001 C CNN
 F 1 "GND" H 8750 5550 50  0000 C CNN
 F 2 "" H 8750 5700 50  0000 C CNN
