File: ModelRocketAvionicsPCB/Sensors.sch (KiCad schematic (older format))
At the start: 17 parts, among them U3 LIS331, U4 L3GD20HTR, U5 MPL3115A2

Commit message: Added Footprints for non-passives
Parts:
- U3: footprint (none) -> Avionics:LIS331HH
- U4: footprint (none) -> Avionics:Gyro_L3GD20HTR
- U5: footprint (none) -> Avionics:MPL3115A2
Changed lines of the file:
@@
 F 0 "U5" H 5800 1750 60  0000 C CNN
 F 1 "MPL3115A2" H 5800 2000 60  0000 C CNN
-F 2 "" H 5800 1600 60  0001 C CNN
+F 2 "Avionics:MPL3115A2" H 5800 1600 60  0001 C CNN
 F 3 "" H 5800 1600 60  0001 C CNN
 F 4 "MPL3115A2-ND" H 5800 1600 60  0001 C CNN "Digi-Key Part Number"
@@
 F 0 "U3" H 5800 3600 60  0000 C CNN
 F 1 "LIS331" H 5800 3700 60  0000 C CNN
-F 2 "" H 5650 3450 60  0001 C CNN
+F 2 "Avionics:LIS331HH" H 5650 3450 60  0001 C CNN
 F 3 "" H 5650 3450 60  0001 C CNN
 F 4 "497-10134-ND" H 5650 3450 60  0001 C CNN "Digi-Key Part Number"
@@
 F 0 "U4" H 5950 5350 60  0000 C CNN
 F 1 "L3GD20HTR" H 5850 5450 60  0000 C CNN
-F 2 "" H 5700 5500 60  0001 C CNN
+F 2 "Avionics:Gyro_L3GD20HTR" H 5700 5500 60  0001 C CNN
 F 3 "" H 5700 5500 60  0001 C CNN
 F 4 "497-13931-1-ND" H 5700 5500 60  0001 C CNN "Digi-Key Part Number"

Commit message: Footprints Completed
Except Jumper Footprints
Parts:
- C19, C20, C21: footprint (none) -> SFUSAT Caps:C_0603; Digi-Key Part Number (none) -> 1276-1871-1-ND; Footprint (none) -> 0603
- C22, C23, C24, C26, C27: footprint (none) -> SFUSAT Caps:C_0402; Digi-Key Part Number (none) -> 587-4552-1-ND; Footprint (none) -> 0402
- C25: footprint (none) -> SFUSAT Caps:C_0603; Digi-Key Part Number (none) -> 490-1543-1-ND; Footprint (none) -> 0603
- C28: footprint (none) -> SFUSAT Caps:C_0402; Digi-Key Part Number (none) -> 478-7867-1-ND; Footprint (none) -> 0402
Changed lines of the file:
@@
 F 0 "C21" H 3425 3600 50  0000 L CNN
 F 1 "10uF" H 3425 3400 50  0000 L CNN
-F 2 "" H 3400 3500 50  0001 C CNN
+F 2 "SFUSAT Caps:C_0603" H 3400 3500 50  0001 C CNN
 F 3 "" H 3400 3500 50  0000 C CNN
+F 4 "1276-1871-1-ND" H 3400 3500 60  0001 C CNN "Digi-Key Part Number"
+F 5 "0603" H 3400 3500 60  0001 C CNN "Footprint"
 	1    3400 3500
 	1    0    0    -1
@@
 F 0 "C24" H 3825 3600 50  0000 L CNN
 F 1 "0.1uF" H 3825 3400 50  0000 L CNN
-F 2 "" H 3838 3350 50  0001 C CNN
+F 2 "SFUSAT Caps:C_0402" H 3838 3350 50  0001 C CNN
 F 3 "" H 3800 3500 50  0000 C CNN
+F 4 "587-4552-1-ND" H 3800 3500 60  0001 C CNN "Digi-Key Part Number"
+F 5 "0402" H 3800 3500 60  0001 C CNN "Footprint"
 	1    3800 3500
 	1    0    0    -1
@@
 F 0 "C27" H 4825 1750 50  0000 L CNN
 F 1 "0.1uF" H 4825 1550 50  0000 L CNN
-F 2 "" H 4838 1500 50  0001 C CNN
+F 2 "SFUSAT Caps:C_0402" H 4838 1500 50  0001 C CNN
 F 3 "" H 4800 1650 50  0000 C CNN
+F 4 "587-4552-1-ND" H 4800 1650 60  0001 C CNN "Digi-Key Part Number"
+F 5 "0402" H 4800 1650 60  0001 C CNN "Footprint"
 	1    4800 1650
 	1    0    0    -1
@@
 F 0 "C19" H 3075 1600 50  0000 L CNN
 F 1 "10uF" H 3075 1400 50  0000 L CNN
-F 2 "" H 3050 1500 50  0001 C CNN
+F 2 "SFUSAT Caps:C_0603" H 3050 1500 50  0001 C CNN
 F 3 "" H 3050 1500 50  0000 C CNN
+F 4 "1276-1871-1-ND" H 3050 1500 60  0001 C CNN "Digi-Key Part Number"
+F 5 "0603" H 3050 1500 60  0001 C CNN "Footprint"
 	1    3050 1500
 	1    0    0    -1
@@
 F 0 "C22" H 3475 1600 50  0000 L CNN
 F 1 "0.1uF" H 3475 1400 50  0000 L CNN
-F 2 "" H 3488 1350 50  0001 C CNN
+F 2 "SFUSAT Caps:C_0402" H 3488 1350 50  0001 C CNN
 F 3 "" H 3450 1500 50  0000 C CNN
+F 4 "587-4552-1-ND" H 3450 1500 60  0001 C CNN "Digi-Key Part Number"
+F 5 "0402" H 3450 1500 60  0001 C CNN "Footprint"
 	1    3450 1500
 	1    0    0    -1
@@
 F 0 "C25" H 3875 1600 50  0000 L CNN
 F 1 "1uF" H 3875 1400 50  0000 L CNN
-F 2 "" H 3888 1350 50  0001 C CNN
+F 2 "SFUSAT Caps:C_0603" H 3888 1350 50  0001 C CNN
 F 3 "" H 3850 1500 50  0000 C CNN
+F 4 "490-1543-1-ND" H 3850 1500 60  0001 C CNN "Digi-Key Part Number"
+F 5 "0603" H 3850 1500 60  0001 C CNN "Footprint"
 	1    3850 1500
 	1    0    0    -1
@@
 F 0 "C28" H 6875 5650 50  0000 L CNN
 F 1 "10nF(25V)" H 6875 5450 50  0000 L CNN
-F 2 "" H 6888 5400 50  0001 C CNN
+F 2 "SFUSAT Caps:C_0402" H 6888 5400 50  0001 C CNN
 F 3 "" H 6850 5550 50  0000 C CNN
+F 4 "478-7867-1-ND" H 6850 5550 60  0001 C CNN "Digi-Key Part Number"
+F 5 "0402" H 6850 5550 60  0001 C CNN "Footprint"
 	1    6850 5550
 	1    0    0    -1
@@
 F 0 "C23" H 3475 5600 50  0000 L CNN
 F 1 ".1uF" H 3475 5400 50  0000 L CNN
-F 2 "" H 3488 5350 50  0001 C CNN
+F 2 "SFUSAT Caps:C_0402" H 3488 5350 50  0001 C CNN
 F 3 "" H 3450 5500 50  0000 C CNN
+F 4 "587-4552-1-ND" H 3450 5500 60  0001 C CNN "Digi-Key Part Number"
+F 5 "0402" H 3450 5500 60  0001 C CNN "Footprint"
 	1    3450 5500
 	1    0    0    -1
@@
 F 0 "C26" H 3875 5600 50  0000 L CNN
 F 1 ".1uF" H 3875 5400 50  0000 L CNN
-F 2 "" H 3888 5350 50  0001 C CNN
+F 2 "SFUSAT Caps:C_0402" H 3888 5350 50  0001 C CNN
 F 3 "" H 3850 5500 50  0000 C CNN
+F 4 "587-4552-1-ND" H 3850 5500 60  0001 C CNN "Digi-Key Part Number"
+F 5 "0402" H 3850 5500 60  0001 C CNN "Footprint"
 	1    3850 5500
 	1    0    0    -1
@@
 F 0 "C20" H 3075 5600 50  0000 L CNN
 F 1 "10uF" H 3075 5400 50  0000 L CNN
-F 2 "" H 3088 5350 50  0001 C CNN
+F 2 "SFUSAT Caps:C_0603" H 3088 5350 50  0001 C CNN
 F 3 "" H 3050 5500 50  0000 C CNN
+F 4 "1276-1871-1-ND" H 3050 5500 60  0001 C CNN "Digi-Key Part Number"
+F 5 "0603" H 3050 5500 60  0001 C CNN "Footprint"
 	1    3050 5500
 	1    0    0    -1

Commit message: Changed polarized caps to use 1206 and digikey part number: 478-10756-1-ND
Parts:
- C19, C21: footprint SFUSAT Caps:C_0603 -> SFUSAT Caps:C_1206; Digi-Key Part Number 1276-1871-1-ND -> 478-10756-1-ND; Footprint 0603 -> (none)
Changed lines of the file:
@@
 F 0 "C21" H 3425 3600 50  0000 L CNN
 F 1 "10uF" H 3425 3400 50  0000 L CNN
-F 2 "SFUSAT Caps:C_0603" H 3400 3500 50  0001 C CNN
+F 2 "SFUSAT Caps:C_1206" H 3400 3500 50  0001 C CNN
 F 3 "" H 3400 3500 50  0000 C CNN
-F 4 "1276-1871-1-ND" H 3400 3500 60  0001 C CNN "Digi-Key Part Number"
-F 5 "0603" H 3400 3500 60  0001 C CNN "Footprint"
+F 4 "478-10756-1-ND" H 3400 3500 60  0001 C CNN "Digi-Key Part Number"
 	1    3400 3500
 	1    0    0    -1
@@
 F 0 "C19" H 3075 1600 50  0000 L CNN
 F 1 "10uF" H 3075 1400 50  0000 L CNN
-F 2 "SFUSAT Caps:C_0603" H 3050 1500 50  0001 C CNN
+F 2 "SFUSAT Caps:C_1206" H 3050 1500 50  0001 C CNN
 F 3 "" H 3050 1500 50  0000 C CNN
-F 4 "1276-1871-1-ND" H 3050 1500 60  0001 C CNN "Digi-Key Part Number"
-F 5 "0603" H 3050 1500 60  0001 C CNN "Footprint"
+F 4 "478-10756-1-ND" H 3050 1500 60  0001 C CNN "Digi-Key Part Number"
 	1    3050 1500
 	1    0    0    -1

Commit message: Began Preliminary Layout
Parts:
- JP1, JP3: footprint (none) -> Avionics:NO_Jumper
- JP2, JP4: footprint (none) -> Avionics:NC_Jumper
Changed lines of the file:
@@
 F 0 "JP2" H 8550 3680 50  0000 C CNN
 F 1 "Jumper_NC_Small" H 8560 3540 50  0001 C CNN
-F 2 "" H 8550 3600 50  0001 C CNN
+F 2 "Avionics:NC_Jumper" H 8550 3600 50  0001 C CNN
 F 3 "" H 8550 3600 50  0000 C CNN
 	1    8550 3600
@@
 F 0 "JP1" H 8550 3380 50  0000 C CNN
 F 1 "Jumper_NO_Small" H 8560 3240 50  0001 C CNN
-F 2 "" H 8550 3300 50  0001 C CNN
+F 2 "Avionics:NO_Jumper" H 8550 3300 50  0001 C CNN
 F 3 "" H 8550 3300 50  0000 C CNN
 	1    8550 3300
@@
 F 0 "JP4" H 8550 5680 50  0000 C CNN
 F 1 "Jumper_NC_Small" H 8560 5540 50  0001 C CNN
-F 2 "" H 8550 5600 50  0001 C CNN
+F 2 "Avionics:NC_Jumper" H 8550 5600 50  0001 C CNN
 F 3 "" H 8550 5600 50  0000 C CNN
 	1    8550 5600
@@
 F 0 "JP3" H 8550 5380 50  0000 C CNN
 F 1 "Jumper_NO_Small" H 8560 5240 50  0001 C CNN
-F 2 "" H 8550 5300 50  0001 C CNN
+F 2 "Avionics:NO_Jumper" H 8550 5300 50  0001 C CNN
 F 3 "" H 8550 5300 50  0000 C CNN
 	1    8550 5300
