File: ModelRocketAvionicsPCB/Sensors.sch (KiCad schematic (older format))
At the start: 17 parts, among them U3 LIS331, U4 L3GD20HTR, U5 MPL3115A2

Commit message: Schematic Check Complete
Parts:
- C28: Footprint 0402 -> (none)
Changed lines of the file:
@@
 F 3 "" H 6850 5550 50  0000 C CNN
 F 4 "478-7867-1-ND" H 6850 5550 60  0001 C CNN "Digi-Key Part Number"
-F 5 "0402" H 6850 5550 60  0001 C CNN "Footprint"
 	1    6850 5550
 	1    0    0    -1

Commit message: Final Board REV 1a - Gerber Files
Parts:
- C20, C25: Footprint 0603 -> (none)
- C22, C23, C24, C26, C27: Footprint 0402 -> (none)
Changed lines of the file:
@@
 F 3 "" H 3800 3500 50  0000 C CNN
 F 4 "587-4552-1-ND" H 3800 3500 60  0001 C CNN "Digi-Key Part Number"
-F 5 "0402" H 3800 3500 60  0001 C CNN "Footprint"
 	1    3800 3500
 	1    0    0    -1
@@
 F 3 "" H 4800 1650 50  0000 C CNN
 F 4 "587-4552-1-ND" H 4800 1650 60  0001 C CNN "Digi-Key Part Number"
-F 5 "0402" H 4800 1650 60  0001 C CNN "Footprint"
 	1    4800 1650
 	1    0    0    -1
@@
 F 3 "" H 3450 1500 50  0000 C CNN
 F 4 "587-4552-1-ND" H 3450 1500 60  0001 C CNN "Digi-Key Part Number"
-F 5 "0402" H 3450 1500 60  0001 C CNN "Footprint"
 	1    3450 1500
 	1    0    0    -1
@@
 F 3 "" H 3850 1500 50  0000 C CNN
 F 4 "490-1543-1-ND" H 3850 1500 60  0001 C CNN "Digi-Key Part Number"
-F 5 "0603" H 3850 1500 60  0001 C CNN "Footprint"
 	1    3850 1500
 	1    0    0    -1
@@
 F 3 "" H 3450 5500 50  0000 C CNN
 F 4 "587-4552-1-ND" H 3450 5500 60  0001 C CNN "Digi-Key Part Number"
-F 5 "0402" H 3450 5500 60  0001 C CNN "Footprint"
 	1    3450 5500
 	1    0    0    -1
@@
 F 3 "" H 3850 5500 50  0000 C CNN
 F 4 "587-4552-1-ND" H 3850 5500 60  0001 C CNN "Digi-Key Part Number"
-F 5 "0402" H 3850 5500 60  0001 C CNN "Footprint"
 	1    3850 5500
 	1    0    0    -1
@@
 F 3 "" H 3050 5500 50  0000 C CNN
 F 4 "1276-1871-1-ND" H 3050 5500 60  0001 C CNN "Digi-Key Part Number"
-F 5 "0603" H 3050 5500 60  0001 C CNN "Footprint"
 	1    3050 5500
 	1    0    0    -1
