File: ModelRocketAvionicsPCB/Power.sch (KiCad schematic (older format))
At the start: 10 parts, among them U6 MCP73831, U7 MIC5219-3.3BM5

Commit message: Added Footprints for non-passives
Parts:
- C31: Digi-Key Part Number (none) -> 490-3296-1-ND
- D1: Digi-Key Part Number (none) -> 160-1447-1-ND
- U6: footprint (none) -> Avionics:MCP73831T-2ACI&slash_OT
- U7: footprint (none) -> Avionics:MIC5219-3.3YM5-TR
Changed lines of the file:
@@
 F 0 "U6" H 3850 3500 60  0000 C CNN
 F 1 "MCP73831" H 3850 3000 60  0000 C CNN
-F 2 "" H 3850 3150 60  0001 C CNN
+F 2 "Avionics:MCP73831T-2ACI&slash_OT" H 3850 3150 60  0001 C CNN
 F 3 "" H 3850 3150 60  0001 C CNN
 F 4 "MCP73831T-2ACI/OTCT-ND" H 3850 3250 60  0001 C CNN "Digi-Key Part Number"
@@
 F 0 "U7" H 7750 3500 60  0000 C CNN
 F 1 "MIC5219-3.3BM5" H 7750 3000 60  0000 C CNN
-F 2 "" H 7750 3150 60  0001 C CNN
+F 2 "Avionics:MIC5219-3.3YM5-TR" H 7750 3150 60  0001 C CNN
 F 3 "" H 7750 3150 60  0001 C CNN
 F 4 "576-1281-1-ND" H 7750 3250 60  0001 C CNN "Digi-Key Part Number"
@@
 F 2 "" V 3300 3500 50  0001 C CNN
 F 3 "" V 3300 3500 50  0000 C CNN
+F 4 "160-1447-1-ND" H 3300 3500 60  0001 C CNN "Digi-Key Part Number"
 	1    3300 3500
 	0    1    1    0
@@
 F 2 "" H 6138 4050 50  0001 C CNN
 F 3 "" H 6100 4200 50  0000 C CNN
+F 4 "490-3296-1-ND" H 6100 4200 60  0001 C CNN "Digi-Key Part Number"
 	1    6100 4200
 	1    0    0    -1

Commit message: Footprints Completed
Except Jumper Footprints
Parts:
- C29, C30: footprint (none) -> SFUSAT Caps:C_0603; Digi-Key Part Number (none) -> 445-7478-1-ND; Footprint (none) -> 0603; Rated Voltage (none) -> 16V
- C31: footprint (none) -> SFUSAT Caps:C_0603
- C32: footprint (none) -> SFUSAT Caps:C_0402; Digi-Key Part Number (none) -> 490-1300-1-ND; Footprint (none) -> 0402
- D1: footprint (none) -> SFUSAT-Res:R_0603
- D2: footprint (none) -> Avionics:B340A; Digi-Key Part Number (none) -> B340A-FDICT-ND
- R13: footprint (none) -> SFUSAT-Res:R_0402; Digi-Key Part Number (none) -> RR05P330DCT-ND
- R14: footprint (none) -> SFUSAT-Res:R_0402; Digi-Key Part Number (none) -> 311-10.0KLRCT-ND
Changed lines of the file:
@@
 F 0 "C29" H 3725 4350 50  0000 L CNN
 F 1 "4.7uF" H 3725 4150 50  0000 L CNN
-F 2 "" H 3738 4100 50  0001 C CNN
+F 2 "SFUSAT Caps:C_0603" H 3738 4100 50  0001 C CNN
 F 3 "" H 3700 4250 50  0000 C CNN
+F 4 "445-7478-1-ND" H 3700 4250 60  0001 C CNN "Digi-Key Part Number"
+F 5 "0603" H 3700 4250 60  0001 C CNN "Footprint"
+F 6 "16V" H 3700 4250 60  0001 C CNN "Rated Voltage"
 	1    3700 4250
 	1    0    0    -1
@@
 F 0 "D2" H 5700 3250 50  0000 C CNN
 F 1 "B340A" H 5700 3050 50  0000 C CNN
-F 2 "" H 5700 3150 50  0001 C CNN
+F 2 "Avionics:B340A" H 5700 3150 50  0001 C CNN
 F 3 "" H 5700 3150 50  0000 C CNN
+F 4 "B340A-FDICT-ND" H 5700 3150 60  0001 C CNN "Digi-Key Part Number"
 	1    5700 3150
 	-1   0    0    1
@@
 F 0 "R14" V 4630 3250 50  0000 C CNN
 F 1 "10k" V 4550 3250 50  0000 C CNN
-F 2 "" V 4480 3250 50  0001 C CNN
+F 2 "SFUSAT-Res:R_0402" V 4480 3250 50  0001 C CNN
 F 3 "" H 4550 3250 50  0000 C CNN
+F 4 "311-10.0KLRCT-ND" V 4550 3250 60  0001 C CNN "Digi-Key Part Number"
 	1    4550 3250
 	0    1    1    0
@@
 F 0 "D1" H 3300 3600 50  0000 L CNN
 F 1 "RED" H 3150 3450 50  0000 L CNN
-F 2 "" V 3300 3500 50  0001 C CNN
+F 2 "SFUSAT-Res:R_0603" V 3300 3500 50  0001 C CNN
 F 3 "" V 3300 3500 50  0000 C CNN
 F 4 "160-1447-1-ND" H 3300 3500 60  0001 C CNN "Digi-Key Part Number"
@@
 F 0 "R13" V 3130 3450 50  0000 C CNN
 F 1 "330" V 3050 3450 50  0000 C CNN
-F 2 "" V 2980 3450 50  0001 C CNN
+F 2 "SFUSAT-Res:R_0402" V 2980 3450 50  0001 C CNN
 F 3 "" H 3050 3450 50  0000 C CNN
+F 4 "RR05P330DCT-ND" V 3050 3450 60  0001 C CNN "Digi-Key Part Number"
 	1    3050 3450
 	-1   0    0    1
@@
 F 0 "C32" H 8325 3650 50  0000 L CNN
 F 1 "470pF" H 8325 3450 50  0000 L CNN
-F 2 "" H 8338 3400 50  0001 C CNN
+F 2 "SFUSAT Caps:C_0402" H 8338 3400 50  0001 C CNN
 F 3 "" H 8300 3550 50  0000 C CNN
+F 4 "490-1300-1-ND" H 8300 3550 60  0001 C CNN "Digi-Key Part Number"
+F 5 "0402" H 8300 3550 60  0001 C CNN "Footprint"
 	1    8300 3550
 	1    0    0    -1
@@
 F 0 "C31" H 6125 4300 50  0000 L CNN
 F 1 "2.2uF" H 6125 4100 50  0000 L CNN
-F 2 "" H 6138 4050 50  0001 C CNN
+F 2 "SFUSAT Caps:C_0603" H 6138 4050 50  0001 C CNN
 F 3 "" H 6100 4200 50  0000 C CNN
 F 4 "490-3296-1-ND" H 6100 4200 60  0001 C CNN "Digi-Key Part Number"
@@
 F 0 "C30" H 4725 4350 50  0000 L CNN
 F 1 "4.7uF" H 4725 4150 50  0000 L CNN
-F 2 "" H 4738 4100 50  0001 C CNN
+F 2 "SFUSAT Caps:C_0603" H 4738 4100 50  0001 C CNN
 F 3 "" H 4700 4250 50  0000 C CNN
+F 4 "445-7478-1-ND" H 4700 4250 60  0001 C CNN "Digi-Key Part Number"
+F 5 "0603" H 4700 4250 60  0001 C CNN "Footprint"
+F 6 "16V" H 4700 4250 60  0001 C CNN "Rated Voltage"
 	1    4700 4250
 	1    0    0    -1
