File: ModelRocketAvionicsPCB/Power.sch (KiCad schematic (older format))
At the start: 10 parts, among them U6 MCP73831, U7 MIC5219-3.3BM5

Commit message: Schematic Check Complete
Parts:
- C31: Digi-Key Part Number 490-3296-1-ND -> 490-10486-6-ND
Changed lines of the file:
@@
 F 2 "SFUSAT Caps:C_0603" H 6138 4050 50  0001 C CNN
 F 3 "" H 6100 4200 50  0000 C CNN
-F 4 "490-3296-1-ND" H 6100 4200 60  0001 C CNN "Digi-Key Part Number"
+F 4 "490-10486-6-ND" H 6100 4200 60  0001 C CNN "Digi-Key Part Number"
 	1    6100 4200
 	1    0    0    -1
