File: ModelRocketAvionicsPCB/AvionicsBoard.sch (KiCad schematic (older format))
At the start: 39 parts, among them CON1 microSD_Card, P1 FTSH-105-01-F-DV, P2 USB_OTG, P3 JST-2, SW1 SW_RST, U1 TM4C123GH6PM, U2 AT25SF161-16Mb_SPI_FLASH, Y1 16Mhz, Y2 32.768kHz

Commit message: oh no
Parts:
- P2: symbol USB_OTG -> USB_OTG-RESCUE-AvionicsBoard
- U1: footprint (none) -> Avionics:TM4C123GH6PMI

Commit message: Added Footprints for non-passives
Parts:
- C10: Digi-Key Part Number (none) -> 490-3296-1-ND
- CON1: footprint (none) -> Avionics:Micro_SD_WM11190CT
- P1: footprint (none) -> Avionics:FTSH-105-01-F-DV-K; Digi-Key Part Number SAM9434-ND -> SAM8796-ND
- P2: footprint (none) -> Avionics:USB_Connector_ZX62-B-5PA; Digi-Key Part Number 609-4053-1-ND -> H125279CT-ND
- P3: footprint (none) -> Avionics:JST_B2B-EH-A(LF)(SN); Digi-Key Part Number (none) -> 455-1611-ND; Header Type (none) -> EH Header
- SW1: footprint (none) -> Avionics:Push_Button_B3S-1000; Digi-Key Part Number (none) -> SW415-ND
- U2: footprint (none) -> Avionics:Flash_Mem_AT25SF161-SSHD
- Y1: footprint (none) -> Avionics:16MHz_Clock; Digi-Key Part Number (none) -> 631-1150-1-ND; Manufacturer Part No (none) -> NX5032GA-16.000000MHZ-LN-CD-1
- Y2: footprint (none) -> Avionics:Crystal_32768Hz_Radial_Can
Changed lines of the file:
@@
 F 0 "P1" H 1300 7500 50  0000 C CNN
 F 1 "FTSH-105-01-F-DV" H 1300 6900 50  0000 C CNN
-F 2 "" H 1300 5950 50  0001 C CNN
+F 2 "Avionics:FTSH-105-01-F-DV-K" H 1300 5950 50  0001 C CNN
 F 3 "" H 1300 5950 50  0000 C CNN
-F 4 "SAM9434-ND" H 1300 7150 60  0001 C CNN "Digi-Key Part Number"
+F 4 "SAM8796-ND" H 1300 7150 60  0001 C CNN "Digi-Key Part Number"
 	1    1300 7150
 	1    0    0    -1
@@
 F 2 "" H 4788 5300 50  0001 C CNN
 F 3 "" H 4750 5450 50  0000 C CNN
+F 4 "490-3296-1-ND" H 4750 5450 60  0001 C CNN "Digi-Key Part Number"
 	1    4750 5450
 	1    0    0    -1
@@
 F 0 "CON1" H 9450 5950 60  0000 C CNN
 F 1 "microSD_Card" H 10200 5500 60  0000 C CNN
-F 2 "" H 9450 5450 60  0001 C CNN
+F 2 "Avionics:Micro_SD_WM11190CT" H 9450 5450 60  0001 C CNN
 F 3 "" H 9450 5450 60  0001 C CNN
 F 4 "WM11190CT-ND" H 9450 5500 60  0001 C CNN "Digi-Key Part Number"
@@
 F 0 "U2" H 8800 4150 60  0000 C CNN
 F 1 "AT25SF161-16Mb_SPI_FLASH" H 9050 3550 60  0000 C CNN
-F 2 "" H 9050 3850 60  0001 C CNN
+F 2 "Avionics:Flash_Mem_AT25SF161-SSHD" H 9050 3850 60  0001 C CNN
 F 3 "" H 9050 3850 60  0001 C CNN
 F 4 "1265-1230-1-ND" H 9050 3850 60  0001 C CNN "Digi-Key Part Number"
@@
 F 0 "P2" H 6825 5175 50  0000 C CNN
 F 1 "USB_OTG" H 6500 5500 50  0000 C CNN
-F 2 "" V 6450 5200 50  0001 C CNN
+F 2 "Avionics:USB_Connector_ZX62-B-5PA" V 6450 5200 50  0001 C CNN
 F 3 "" V 6450 5200 50  0000 C CNN
-F 4 "609-4053-1-ND" H 6500 5300 60  0001 C CNN "Digi-Key Part Number"
+F 4 "H125279CT-ND" H 6500 5300 60  0001 C CNN "Digi-Key Part Number"
 	1    6500 5300
 	0    1    1    0
@@
 F 0 "Y2" H 10050 2500 50  0000 C CNN
 F 1 "32.768kHz" H 10050 2200 50  0000 C CNN
-F 2 "" H 10050 2350 50  0001 C CNN
+F 2 "Avionics:Crystal_32768Hz_Radial_Can" H 10050 2350 50  0001 C CNN
 F 3 "" H 10050 2350 50  0000 C CNN
 	1    10050 2350
@@
 F 0 "Y1" H 9100 2300 50  0000 C CNN
 F 1 "16Mhz" H 9100 2000 50  0000 C CNN
-F 2 "" H 9100 2150 50  0001 C CNN
+F 2 "Avionics:16MHz_Clock" H 9100 2150 50  0001 C CNN
 F 3 "" H 9100 2150 50  0000 C CNN
+F 4 "631-1150-1-ND" H 9100 2150 60  0001 C CNN "Digi-Key Part Number"
+F 5 "NX5032GA-16.000000MHZ-LN-CD-1" H 9100 2150 60  0001 C CNN "Manufacturer Part No"
 	1    9100 2150
 	0    -1   -1   0
@@
 F 0 "SW1" H 6100 3860 50  0000 C CNN
 F 1 "SW_RST" H 5950 3670 50  0000 C CNN
-F 2 "" H 5950 3750 50  0001 C CNN
+F 2 "Avionics:Push_Button_B3S-1000" H 5950 3750 50  0001 C CNN
 F 3 "" H 5950 3750 50  0000 C CNN
+F 4 "SW415-ND" H 5950 3750 60  0001 C CNN "Digi-Key Part Number"
 	1    5950 3750
 	1    0    0    -1
@@
 F 0 "P3" H 10850 1000 50  0000 C CNN
 F 1 "JST-2" H 10850 1300 50  0000 C CNN
-F 2 "" H 10850 1150 50  0001 C CNN
+F 2 "Avionics:JST_B2B-EH-A(LF)(SN)" H 10850 1150 50  0001 C CNN
 F 3 "" H 10850 1150 50  0000 C CNN
+F 4 "455-1611-ND" H 10850 1150 60  0001 C CNN "Digi-Key Part Number"
+F 5 "EH Header" H 10850 1150 60  0001 C CNN "Header Type"
 	1    10850 1150
 	1    0    0    -1

Commit message: Footprints Completed
Except Jumper Footprints
Parts:
- C1, C5: footprint (none) -> SFUSAT Caps:C_0402; Digi-Key Part Number (none) -> 478-7867-1-ND; Footprint (none) -> 0402
- C10: footprint (none) -> SFUSAT Caps:C_0603
- C11, C12, C13, C6, C9: footprint (none) -> SFUSAT Caps:C_0603; Digi-Key Part Number (none) -> 490-1543-1-ND; Footprint (none) -> 0603
- C14, C2, C7, C8: footprint (none) -> SFUSAT Caps:C_0402; Digi-Key Part Number (none) -> 587-4552-1-ND; Footprint (none) -> 0402
- C15, C16: footprint (none) -> SFUSAT Caps:C_0402; Digi-Key Part Number (none) -> 712-1252-1-ND; Footprint (none) -> 0402
- C17: footprint (none) -> SFUSAT Caps:C_0402; Digi-Key Part Number (none) -> 478-10149-1-ND; Footprint (none) -> 0402
- C18: footprint (none) -> SFUSAT Caps:C_0402
- C3: footprint (none) -> SFUSAT Caps:C_0402; Digi-Key Part Number (none) -> 478-7867-1-ND
- C4: footprint (none) -> SFUSAT Caps:C_0402; Digi-Key Part Number (none) -> 587-4552-1-ND
- R1: footprint (none) -> SFUSAT-Res:R_0402; Digi-Key Part Number (none) -> P100DECT-ND
- R10, R11, R12, R2, R3, R4, R7, R8, R9: footprint (none) -> SFUSAT-Res:R_0402; Digi-Key Part Number (none) -> 311-10.0KLRCT-ND
- R5, R6: footprint (none) -> SFUSAT-Res:R_0402; Digi-Key Part Number (none) -> P4.7KDCCT-ND
Changed lines of the file:
@@
 F 0 "R5" V 3730 6700 50  0000 C CNN
 F 1 "4.7k" V 3650 6700 50  0000 C CNN
-F 2 "" V 3580 6700 50  0001 C CNN
+F 2 "SFUSAT-Res:R_0402" V 3580 6700 50  0001 C CNN
 F 3 "" H 3650 6700 50  0001 C CNN
+F 4 "P4.7KDCCT-ND" V 3650 6700 60  0001 C CNN "Digi-Key Part Number"
 	1    3650 6700
 	1    0    0    -1
@@
 F 0 "R6" V 3930 6700 50  0000 C CNN
 F 1 "4.7k" V 3850 6700 50  0000 C CNN
-F 2 "" V 3780 6700 50  0001 C CNN
+F 2 "SFUSAT-Res:R_0402" V 3780 6700 50  0001 C CNN
 F 3 "" H 3850 6700 50  0001 C CNN
+F 4 "P4.7KDCCT-ND" V 3850 6700 60  0001 C CNN "Digi-Key Part Number"
 	1    3850 6700
 	1    0    0    -1
@@
 F 0 "R1" V 880 6650 50  0000 C CNN
 F 1 "100" V 800 6650 50  0000 C CNN
-F 2 "" V 730 6650 50  0001 C CNN
+F 2 "SFUSAT-Res:R_0402" V 730 6650 50  0001 C CNN
 F 3 "" H 800 6650 50  0000 C CNN
+F 4 "P100DECT-ND" V 800 6650 60  0001 C CNN "Digi-Key Part Number"
 	1    800  6650
 	1    0    0    -1
@@
 F 0 "R2" V 1830 6650 50  0000 C CNN
 F 1 "10k" V 1750 6650 50  0000 C CNN
-F 2 "" V 1680 6650 50  0001 C CNN
+F 2 "SFUSAT-Res:R_0402" V 1680 6650 50  0001 C CNN
 F 3 "" H 1750 6650 50  0000 C CNN
+F 4 "311-10.0KLRCT-ND" V 1750 6650 60  0001 C CNN "Digi-Key Part Number"
 	1    1750 6650
 	1    0    0    -1
@@
 F 0 "R4" V 2030 6650 50  0000 C CNN
 F 1 "10k" V 1950 6650 50  0000 C CNN
-F 2 "" V 1880 6650 50  0001 C CNN
+F 2 "SFUSAT-Res:R_0402" V 1880 6650 50  0001 C CNN
 F 3 "" H 1950 6650 50  0000 C CNN
+F 4 "311-10.0KLRCT-ND" V 1950 6650 60  0001 C CNN "Digi-Key Part Number"
 	1    1950 6650
 	1    0    0    -1
@@
 F 0 "R3" V 1830 7550 50  0000 C CNN
 F 1 "10k" V 1750 7550 50  0000 C CNN
-F 2 "" V 1680 7550 50  0001 C CNN
+F 2 "SFUSAT-Res:R_0402" V 1680 7550 50  0001 C CNN
 F 3 "" H 1750 7550 50  0000 C CNN
+F 4 "311-10.0KLRCT-ND" V 1750 7550 60  0001 C CNN "Digi-Key Part Number"
 	1    1750 7550
 	1    0    0    -1
@@
 F 0 "C1" H 1225 5550 50  0000 L CNN
 F 1 "0.01uF" H 1225 5350 50  0000 L CNN
-F 2 "" H 1238 5300 50  0001 C CNN
+F 2 "SFUSAT Caps:C_0402" H 1238 5300 50  0001 C CNN
 F 3 "" H 1200 5450 50  0000 C CNN
+F 4 "478-7867-1-ND" H 1200 5450 60  0001 C CNN "Digi-Key Part Number"
+F 5 "0402" H 1200 5450 60  0001 C CNN "Footprint"
 	1    1200 5450
 	1    0    0    -1
@@
 F 0 "C2" H 1575 5550 50  0000 L CNN
 F 1 "0.1uF" H 1575 5350 50  0000 L CNN
-F 2 "" H 1588 5300 50  0001 C CNN
+F 2 "SFUSAT Caps:C_0402" H 1588 5300 50  0001 C CNN
 F 3 "" H 1550 5450 50  0000 C CNN
+F 4 "587-4552-1-ND" H 1550 5450 60  0001 C CNN "Digi-Key Part Number"
+F 5 "0402" H 1550 5450 60  0001 C CNN "Footprint"
 	1    1550 5450
 	1    0    0    -1
@@
 F 0 "C3" H 1925 5550 50  0000 L CNN
 F 1 "0.01uF" H 1925 5350 50  0000 L CNN
-F 2 "" H 1938 5300 50  0001 C CNN
+F 2 "SFUSAT Caps:C_0402" H 1938 5300 50  0001 C CNN
 F 3 "" H 1900 5450 50  0000 C CNN
+F 4 "478-7867-1-ND" H 1900 5450 60  0001 C CNN "Digi-Key Part Number"
 	1    1900 5450
 	1    0    0    -1
@@
 F 0 "C4" H 2275 5550 50  0000 L CNN
 F 1 "0.1uF" H 2275 5350 50  0000 L CNN
-F 2 "" H 2288 5300 50  0001 C CNN
+F 2 "SFUSAT Caps:C_0402" H 2288 5300 50  0001 C CNN
 F 3 "" H 2250 5450 50  0000 C CNN
+F 4 "587-4552-1-ND" H 2250 5450 60  0001 C CNN "Digi-Key Part Number"
 	1    2250 5450
 	1    0    0    -1
@@
 F 0 "C5" H 2625 5550 50  0000 L CNN
 F 1 "0.01uF" H 2625 5350 50  0000 L CNN
-F 2 "" H 2638 5300 50  0001 C CNN
+F 2 "SFUSAT Caps:C_0402" H 2638 5300 50  0001 C CNN
 F 3 "" H 2600 5450 50  0000 C CNN
+F 4 "478-7867-1-ND" H 2600 5450 60  0001 C CNN "Digi-Key Part Number"
+F 5 "0402" H 2600 5450 60  0001 C CNN "Footprint"
 	1    2600 5450
 	1    0    0    -1
@@
 F 0 "C6" H 2975 5550 50  0000 L CNN
 F 1 "1uF" H 2975 5350 50  0000 L CNN
-F 2 "" H 2988 5300 50  0001 C CNN
+F 2 "SFUSAT Caps:C_0603" H 2988 5300 50  0001 C CNN
 F 3 "" H 2950 5450 50  0000 C CNN
+F 4 "490-1543-1-ND" H 2950 5450 60  0001 C CNN "Digi-Key Part Number"
+F 5 "0603" H 2950 5450 60  0001 C CNN "Footprint"
 	1    2950 5450
 	1    0    0    -1
@@
 F 0 "C7" H 3925 5550 50  0000 L CNN
 F 1 "0.1uF" H 3925 5350 50  0000 L CNN
-F 2 "" H 3938 5300 50  0001 C CNN
+F 2 "SFUSAT Caps:C_0402" H 3938 5300 50  0001 C CNN
 F 3 "" H 3900 5450 50  0000 C CNN
+F 4 "587-4552-1-ND" H 3900 5450 60  0001 C CNN "Digi-Key Part Number"
+F 5 "0402" H 3900 5450 60  0001 C CNN "Footprint"
 	1    3900 5450
 	1    0    0    -1
@@
 F 0 "C8" H 4225 5550 50  0000 L CNN
 F 1 "0.1uF" H 4225 5350 50  0000 L CNN
-F 2 "" H 4238 5300 50  0001 C CNN
+F 2 "SFUSAT Caps:C_0402" H 4238 5300 50  0001 C CNN
 F 3 "" H 4200 5450 50  0000 C CNN
+F 4 "587-4552-1-ND" H 4200 5450 60  0001 C CNN "Digi-Key Part Number"
+F 5 "0402" H 4200 5450 60  0001 C CNN "Footprint"
 	1    4200 5450
 	1    0    0    -1
@@
 F 0 "C9" H 4525 5550 50  0000 L CNN
 F 1 "1uF" H 4525 5350 50  0000 L CNN
-F 2 "" H 4538 5300 50  0001 C CNN
+F 2 "SFUSAT Caps:C_0603" H 4538 5300 50  0001 C CNN
 F 3 "" H 4500 5450 50  0000 C CNN
+F 4 "490-1543-1-ND" H 4500 5450 60  0001 C CNN "Digi-Key Part Number"
+F 5 "0603" H 4500 5450 60  0001 C CNN "Footprint"
 	1    4500 5450
 	1    0    0    -1
@@
 F 0 "C10" H 4775 5550 50  0000 L CNN
 F 1 "2.2uF" H 4775 5350 50  0000 L CNN
-F 2 "" H 4788 5300 50  0001 C CNN
+F 2 "SFUSAT Caps:C_0603" H 4788 5300 50  0001 C CNN
 F 3 "" H 4750 5450 50  0000 C CNN
 F 4 "490-3296-1-ND" H 4750 5450 60  0001 C CNN "Digi-Key Part Number"
@@
 F 0 "R11" V 8730 6050 50  0000 C CNN
 F 1 "10k" V 8650 6050 50  0000 C CNN
-F 2 "" V 8580 6050 50  0001 C CNN
+F 2 "SFUSAT-Res:R_0402" V 8580 6050 50  0001 C CNN
 F 3 "" H 8650 6050 50  0000 C CNN
+F 4 "311-10.0KLRCT-ND" V 8650 6050 60  0001 C CNN "Digi-Key Part Number"
 	1    8650 6050
 	1    0    0    -1
@@
 F 0 "R10" V 8730 4900 50  0000 C CNN
 F 1 "10k" V 8650 4900 50  0000 C CNN
-F 2 "" V 8580 4900 50  0001 C CNN
+F 2 "SFUSAT-Res:R_0402" V 8580 4900 50  0001 C CNN
 F 3 "" H 8650 4900 50  0000 C CNN
+F 4 "311-10.0KLRCT-ND" V 8650 4900 60  0001 C CNN "Digi-Key Part Number"
 	1    8650 4900
 	1    0    0    -1
@@
 F 0 "R9" V 8530 4900 50  0000 C CNN
 F 1 "10k" V 8450 4900 50  0000 C CNN
-F 2 "" V 8380 4900 50  0001 C CNN
+F 2 "SFUSAT-Res:R_0402" V 8380 4900 50  0001 C CNN
 F 3 "" H 8450 4900 50  0000 C CNN
+F 4 "311-10.0KLRCT-ND" V 8450 4900 60  0001 C CNN "Digi-Key Part Number"
 	1    8450 4900
 	1    0    0    -1
@@
 F 0 "C14" H 7325 5600 50  0000 L CNN
 F 1 "0.1uF" H 7325 5400 50  0000 L CNN
-F 2 "" H 7338 5350 50  0001 C CNN
+F 2 "SFUSAT Caps:C_0402" H 7338 5350 50  0001 C CNN
 F 3 "" H 7300 5500 50  0000 C CNN
+F 4 "587-4552-1-ND" H 7300 5500 60  0001 C CNN "Digi-Key Part Number"
+F 5 "0402" H 7300 5500 60  0001 C CNN "Footprint"
 	1    7300 5500
 	1    0    0    -1
@@
 F 0 "R12" V 9980 3600 50  0000 C CNN
 F 1 "10k" V 9900 3600 50  0000 C CNN
-F 2 "" V 9830 3600 50  0001 C CNN
+F 2 "SFUSAT-Res:R_0402" V 9830 3600 50  0001 C CNN
 F 3 "" H 9900 3600 50  0000 C CNN
+F 4 "311-10.0KLRCT-ND" V 9900 3600 60  0001 C CNN "Digi-Key Part Number"
 	1    9900 3600
 	1    0    0    -1
@@
 F 0 "R8" V 7780 3700 50  0000 C CNN
 F 1 "10k" V 7700 3700 50  0000 C CNN
-F 2 "" V 7630 3700 50  0001 C CNN
+F 2 "SFUSAT-Res:R_0402" V 7630 3700 50  0001 C CNN
 F 3 "" H 7700 3700 50  0000 C CNN
+F 4 "311-10.0KLRCT-ND" V 7700 3700 60  0001 C CNN "Digi-Key Part Number"
 	1    7700 3700
 	1    0    0    -1
@@
 F 0 "C11" H 6025 4500 50  0000 L CNN
 F 1 "1uF" H 6025 4300 50  0000 L CNN
-F 2 "" H 6038 4250 50  0001 C CNN
+F 2 "SFUSAT Caps:C_0603" H 6038 4250 50  0001 C CNN
 F 3 "" H 6000 4400 50  0000 C CNN
+F 4 "490-1543-1-ND" H 6000 4400 60  0001 C CNN "Digi-Key Part Number"
+F 5 "0603" H 6000 4400 60  0001 C CNN "Footprint"
 	1    6000 4400
 	1    0    0    -1
@@
 F 0 "C12" H 6325 4500 50  0000 L CNN
 F 1 "1uF" H 6325 4300 50  0000 L CNN
-F 2 "" H 6338 4250 50  0001 C CNN
+F 2 "SFUSAT Caps:C_0603" H 6338 4250 50  0001 C CNN
 F 3 "" H 6300 4400 50  0000 C CNN
+F 4 "490-1543-1-ND" H 6300 4400 60  0001 C CNN "Digi-Key Part Number"
+F 5 "0603" H 6300 4400 60  0001 C CNN "Footprint"
 	1    6300 4400
 	1    0    0    -1
@@
 F 0 "C13" H 6625 4500 50  0000 L CNN
 F 1 "1uF" H 6625 4300 50  0000 L CNN
-F 2 "" H 6638 4250 50  0001 C CNN
+F 2 "SFUSAT Caps:C_0603" H 6638 4250 50  0001 C CNN
 F 3 "" H 6600 4400 50  0000 C CNN
+F 4 "490-1543-1-ND" H 6600 4400 60  0001 C CNN "Digi-Key Part Number"
+F 5 "0603" H 6600 4400 60  0001 C CNN "Footprint"
 	1    6600 4400
 	1    0    0    -1
@@
 F 0 "C15" H 8725 2650 50  0000 L CNN
 F 1 "10pF" H 8725 2450 50  0000 L CNN
-F 2 "" H 8738 2400 50  0001 C CNN
+F 2 "SFUSAT Caps:C_0402" H 8738 2400 50  0001 C CNN
 F 3 "" H 8700 2550 50  0000 C CNN
+F 4 "712-1252-1-ND" H 8700 2550 60  0001 C CNN "Digi-Key Part Number"
+F 5 "0402" H 8700 2550 60  0001 C CNN "Footprint"
 	1    8700 2550
 	1    0    0    -1
@@
 F 0 "C16" H 9125 2650 50  0000 L CNN
 F 1 "10pF" H 9125 2450 50  0000 L CNN
-F 2 "" H 9138 2400 50  0001 C CNN
+F 2 "SFUSAT Caps:C_0402" H 9138 2400 50  0001 C CNN
 F 3 "" H 9100 2550 50  0000 C CNN
+F 4 "712-1252-1-ND" H 9100 2550 60  0001 C CNN "Digi-Key Part Number"
+F 5 "0402" H 9100 2550 60  0001 C CNN "Footprint"
 	1    9100 2550
 	1    0    0    -1
@@
 F 0 "C18" H 10375 2650 50  0000 L CNN
 F 1 "24pF" H 10375 2450 50  0000 L CNN
-F 2 "" H 10388 2400 50  0001 C CNN
+F 2 "SFUSAT Caps:C_0402" H 10388 2400 50  0001 C CNN
 F 3 "" H 10350 2550 50  0000 C CNN
 	1    10350 2550
@@
 F 0 "C17" H 10375 2250 50  0000 L CNN
 F 1 "24pF" H 10375 2050 50  0000 L CNN
-F 2 "" H 10388 2000 50  0001 C CNN
+F 2 "SFUSAT Caps:C_0402" H 10388 2000 50  0001 C CNN
 F 3 "" H 10350 2150 50  0000 C CNN
+F 4 "478-10149-1-ND" H 10350 2150 60  0001 C CNN "Digi-Key Part Number"
+F 5 "0402" H 10350 2150 60  0001 C CNN "Footprint"
 	1    10350 2150
 	1    0    0    -1
@@
 F 0 "R7" V 6430 3550 50  0000 C CNN
 F 1 "10k" V 6350 3550 50  0000 C CNN
-F 2 "" V 6280 3550 50  0001 C CNN
+F 2 "SFUSAT-Res:R_0402" V 6280 3550 50  0001 C CNN
 F 3 "" H 6350 3550 50  0000 C CNN
+F 4 "311-10.0KLRCT-ND" V 6350 3550 60  0001 C CNN "Digi-Key Part Number"
 	1    6350 3550
 	1    0    0    -1

Commit message: Completed Preliminary Layout
Parts:
- Y2: Digi-Key Part Number (none) -> 535-9034-ND
Connections:
- net PB7/ACC_INT2: now reaches U1.4 (PB7)
- net PF4/GYR_INT1: now reaches U1.5 (PF4)
- net PB5/BAR_INT1: now reaches U1.57 (PB5)
- net PB4/BAR_INT2: now reaches U1.58 (PB4)
- net PE3/GYR_INT2/DRDY: now reaches U1.6 (PE3)
- net PE2/GYR_DEN: now reaches U1.7 (PE2)
Changed lines of the file:
@@
 F 2 "Avionics:Crystal_32768Hz_Radial_Can" H 10050 2350 50  0001 C CNN
 F 3 "" H 10050 2350 50  0000 C CNN
+F 4 "535-9034-ND" H 10050 2350 60  0001 C CNN "Digi-Key Part Number"
 	1    10050 2350
 	0    -1   -1   0
@@
 Wire Wire Line
 	2200 1300 2200 1250
+Text GLabel 1400 2450 0    60   Input ~ 0
+PB7/ACC_INT2
+Wire Wire Line
+	1450 2450 1400 2450
+Text GLabel 1400 2150 0    60   Input ~ 0
+PB6/ACC_INT1
+Text GLabel 1400 2550 0    60   Input ~ 0
+PF4/GYR_INT1
+Text GLabel 1400 2650 0    60   Input ~ 0
+PE3/GYR_INT2/DRDY
+Text GLabel 1400 2750 0    60   Input ~ 0
+PE2/GYR_DEN
+Wire Wire Line
+	1400 2550 1450 2550
+Wire Wire Line
+	1450 2650 1400 2650
+Wire Wire Line
+	1400 2750 1450 2750
+Text GLabel 2600 1250 1    60   Input ~ 0
+PB5/BAR_INT1
+Text GLabel 2500 1250 1    60   Input ~ 0
+PB4/BAR_INT2
+Wire Wire Line
+	2600 1300 2600 1250
+Wire Wire Line
+	2500 1300 2500 1250
+Text GLabel 3975 7400 0    60   Input ~ 0
+PE2/GYR_DEN
+Text GLabel 5675 7500 2    60   Input ~ 0
+PE3/GYR_INT2/DRDY
+Text GLabel 5675 7400 2    60   Input ~ 0
+PF4/GYR_INT1
+Text GLabel 5675 7000 2    60   Input ~ 0
+PB7/ACC_INT2
+Text GLabel 5675 6900 2    60   Input ~ 0
+PB6/ACC_INT1
+Text GLabel 5675 7250 2    60   Input ~ 0
+PB4/BAR_INT2
+Text GLabel 5675 7150 2    60   Input ~ 0
+PB5/BAR_INT1
+Wire Wire Line
+	4000 7400 4050 7400
+Wire Wire Line
+	5600 7500 5675 7500
+Wire Wire Line
+	5675 7400 5600 7400
+Wire Wire Line
+	5675 7250 5600 7250
+Wire Wire Line
+	5600 7150 5675 7150
+Wire Wire Line
+	5675 7000 5600 7000
+Wire Wire Line
+	5600 6900 5675 6900
 $EndSCHEMATC

Commit message: Partially Complete Updated Avionics Layout
Final Pinout and Silk Screen still needs to be completed.
Parts:
- added U8, U9: CONNHeaderFemale16, Avionics:16x1_Female_Header, symbol CONNHeaderFemale16
Connections:
- net PB6/ACC_INT1: now also U1.1 (PB6)
- net PE2/GYR_DEN: now also U1.5 (PF4); no longer U1.7 (PE2)
- net PE3/GYR_INT2/DRDY: now also U1.7 (PE2); no longer U1.6 (PE3)
- net PF4/GYR_INT1: now also U1.6 (PE3); no longer U1.5 (PF4)
Other:
- note added: "Left Side Female Header"
- note added: "Right Side Female Header\n"
