File: ModelRocketAvionicsPCB/AvionicsBoard.sch (KiCad schematic (older format))
At the start: 41 parts, among them CON1 microSD_Card, P1 FTSH-105-01-F-DV, P2 USB_OTG, P3 JST-2, SW1 SW_RST, U1 TM4C123GH6PM, U2 AT25SF161-16Mb_SPI_FLASH, U8 CONNHeaderFemale16, U9 CONNHeaderFemale16, Y1 16Mhz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

Commit message: Updated Sch
Parts:
- added D3: Led_Small, SFUSAT-Res:R_0603, symbol Led_Small
- added R15: 330, SFUSAT-Res:R_0402, symbol R
Connections:
- net PB4/BAR_INT2 is gone; now on net PB4: U1.58 (PB4)
- net PB5/BAR_INT1 is gone; now on net PB5: U1.57 (PB5)
- net PC1/JTAG_TCK is gone; now on net PC0/JTAG_TCK: U1.52 (PC0/TCK/SWCLK)
- net +3V3: now also U8.3, U8.4, U9.16
- net GND: now also R3.2, U8.16, U9.1, U9.2, D3.1 (K)
- net PB2/I2C_SCL: now also U9.3
- net PB3/I2C_SDA: now also U9.4
- net PD0/SSI1CLK: now also U9.12
- net PD1/SSI1Fss: now also U9.13
- net PD2/SSI1Rx: now also U9.14
- net PD3/SSI1Tx: now also U9.15
- net RESET: now also U9.6
- net WAKE: now also U8.5
- net PD7: now reaches U1.10 (PD7)
- net PD7: now also U8.14
- net PC7: now reaches U1.13 (PC7)
- net PC7: now also U8.13
- net PC6: now reaches U1.14 (PC6)
- net PC6: now also U8.12
- net PC5: now reaches U1.15 (PC5)
- net PC5: now also U8.11
- net PC4: now reaches U1.16 (PC4)
- net PC4: now also U8.10
- net PA0/U0Rx: now reaches U1.17 (PA0/U0Rx)
- net PA0/U0Rx: now also U8.9
- net PA1/U0Tx: now reaches U1.18 (PA1/U0Tx)
- net PA1/U0Tx: now also U8.8
- net PA6: now reaches U1.23 (PA6)
- net PA6: now also U8.7
- net PA7: now reaches U1.24 (PA7)
- net PA7: now also U8.6
- net PF0: now reaches U1.28 (PF0)
- net PF1: now reaches U1.29 (PF1)
- net PF2/BAR_INT1: now reaches U1.30 (PF2)
- net PF3/BAR_INT2: now reaches U1.31 (PF3)
- net HIB: now reaches U1.33 (HIB)
- net HIB: now also U9.7
- net PD6: now reaches U1.53 (PD6)
- net PD6: now also U9.5
- net PE4: now reaches U1.59 (PE4)
- net PE4: now also U9.10
- net PE5: now reaches U1.60 (PE5)
- net PE5: now also U9.11
- net PE1/IND_LED: now reaches U1.8 (PE1)
- net PE1/IND_LED: now also R15.2
- net PE0: now reaches U1.9 (PE0)
- net PE0: now also U8.15
- net +VBAT: now reaches U8.1
- net +VBAT: now also U8.2
- net PB5: now reaches U9.8
- net PB4: now reaches U9.9
- net PB6/ACC_INT1 renamed PB6/GYR_INT2/DRDY
- net PB7/ACC_INT2 renamed PB7/GYR_INT1
- net PD4/USB0_DM renamed USB0_D-
- net PD5/USB0_DP renamed USB0_D+
- net PE2/GYR_DEN renamed PF4/GYR_DEN
- net PE3/GYR_INT2/DRDY renamed PE2/ACC_INT2
- net PF4/GYR_INT1 renamed PE3/ACC_INT1
- net Power/+VBAT renamed Power Switch/+VBAT
- new net: D3.2 (A), R15.1
Other:
- note added: "Indicator LED"
- note added: "Left Side Female Header\n"
- note added: "Power Switch - Slide Switch and P-MOSFET"
- note added: "Right Side Female Header"
- note removed: "Left Side Female Header"
- note removed: "Right Side Female Header\n"
- moved on the sheet: P3, U8

Commit message: Schematic Check Complete
Parts:
- R15: value 330 -> 100; Digi-Key Part Number RR05P330DCT-ND -> P100DECT-ND
Other:
- moved on the sheet: U8, U9
Changed lines of the file:
@@
 L CONNHeaderFemale16 U8
 U 1 1 5B41BDEB
-P 6850 1700
-F 0 "U8" H 6850 800 60  0000 C CNN
-F 1 "CONNHeaderFemale16" H 6700 2525 60  0000 C CNN
-F 2 "Avionics:16x1_Female_Header" H 6600 1550 60  0001 C CNN
-F 3 "" H 6600 1550 60  0001 C CNN
-	1    6850 1700
+P 7000 1700
+F 0 "U8" H 7000 800 60  0000 C CNN
+F 1 "CONNHeaderFemale16" H 6675 2525 60  0000 C CNN
+F 2 "Avionics:16x1_Female_Header" H 6750 1550 60  0001 C CNN
+F 3 "" H 6750 1550 60  0001 C CNN
+	1    7000 1700
 	1    0    0    -1
 $EndComp
@@
 L CONNHeaderFemale16 U9
 U 1 1 5B41BEC2
-P 8100 1725
-F 0 "U9" H 8100 825 60  0000 C CNN
-F 1 "CONNHeaderFemale16" H 7975 2550 60  0000 C CNN
-F 2 "Avionics:16x1_Female_Header" H 7850 1575 60  0001 C CNN
-F 3 "" H 7850 1575 60  0001 C CNN
-	1    8100 1725
+P 8325 1725
+F 0 "U9" H 8325 825 60  0000 C CNN
+F 1 "CONNHeaderFemale16" H 7950 2575 60  0000 C CNN
+F 2 "Avionics:16x1_Female_Header" H 8075 1575 60  0001 C CNN
+F 3 "" H 8075 1575 60  0001 C CNN
+	1    8325 1725
 	1    0    0    -1
 $EndComp
@@
 P 5325 1875
 F 0 "R15" V 5405 1875 50  0000 C CNN
-F 1 "330" V 5325 1875 50  0000 C CNN
+F 1 "100" V 5325 1875 50  0000 C CNN
 F 2 "SFUSAT-Res:R_0402" V 5255 1875 50  0001 C CNN
 F 3 "" H 5325 1875 50  0000 C CNN
-F 4 "RR05P330DCT-ND" V 5325 1875 60  0001 C CNN "Digi-Key Part Number"
+F 4 "P100DECT-ND" V 5325 1875 60  0001 C CNN "Digi-Key Part Number"
 	1    5325 1875
 	1    0    0    -1
@@
 	3975 7400 4050 7400
 Wire Notes Line
-	8500 500  8500 3050
-Wire Notes Line
-	8500 3050 7250 3050
-Wire Notes Line
-	7250 3050 7250 500
-Wire Notes Line
-	7250 500  8500 500
-Wire Notes Line
-	7200 500  7200 3050
-Wire Notes Line
-	7200 3050 6000 3050
+	8500 3050 8500 500
+Wire Notes Line
+	6000 3050 7200 3050
 Wire Notes Line
 	6000 3050 6000 500
@@
 	5325 2025 5325 2075
 Wire Wire Line
-	6550 2500 6600 2500
+	6700 2500 6750 2500
 Wire Wire Line
 	1750 7700 1750 7725
@@
 Wire Wire Line
 	3950 3650 4000 3650
-Text GLabel 6550 1000 0    60   Input ~ 0
+Text GLabel 6700 1000 0    60   Input ~ 0
 +VBAT
-Text GLabel 6550 1100 0    60   Input ~ 0
+Text GLabel 6700 1100 0    60   Input ~ 0
 +VBAT
-Text GLabel 6550 1200 0    60   Input ~ 0
+Text GLabel 6700 1200 0    60   Input ~ 0
 PWR_VDD
-Text GLabel 6550 1300 0    60   Input ~ 0
+Text GLabel 6700 1300 0    60   Input ~ 0
 PWR_VDD
-Text GLabel 6550 1400 0    60   Input ~ 0
+Text GLabel 6700 1400 0    60   Input ~ 0
 WAKE
-Text GLabel 6550 1500 0    60   Input ~ 0
+Text GLabel 6700 1500 0    60   Input ~ 0
 PA7
-Text GLabel 6550 1600 0    60   Input ~ 0
+Text GLabel 6700 1600 0    60   Input ~ 0
 PA6
-Text GLabel 6550 1700 0    60   Input ~ 0
+Text GLabel 6700 1700 0    60   Input ~ 0
 PA1/U0Tx
-Text GLabel 6550 1800 0    60   Input ~ 0
+Text GLabel 6700 1800 0    60   Input ~ 0
 PA0/U0Rx
-Text GLabel 6550 1900 0    60   Input ~ 0
+Text GLabel 6700 1900 0    60   Input ~ 0
 PC4
-Text GLabel 6550 2000 0    60   Input ~ 0
+Text GLabel 6700 2000 0    60   Input ~ 0
 PC5
-Text GLabel 6550 2100 0    60   Input ~ 0
+Text GLabel 6700 2100 0    60   Input ~ 0
 PC6
-Text GLabel 6550 2300 0    60   Input ~ 0
+Text GLabel 6700 2300 0    60   Input ~ 0
 PD7
-Text GLabel 6550 2400 0    60   Input ~ 0
+Text GLabel 6700 2400 0    60   Input ~ 0
 PE0
-Text GLabel 6550 2500 0    60   Input ~ 0
+Text GLabel 6700 2500 0    60   Input ~ 0
 PWR_GND
 Wire Wire Line
@@
 	2500 3950 2500 4000
 Wire Wire Line
-	6550 2400 6600 2400
-Wire Wire Line
-	6600 2300 6550 2300
-Wire Wire Line
-	6550 2200 6600 2200
-Wire Wire Line
-	6600 2100 6550 2100
-Wire Wire Line
-	6550 2000 6600 2000
-Wire Wire Line
-	6550 1900 6600 1900
-Wire Wire Line
-	6600 1800 6550 1800
-Wire Wire Line
-	6550 1700 6600 1700
-Wire Wire Line
-	6600 1600 6550 1600
-Wire Wire Line
-	6550 1500 6600 1500
-Wire Wire Line
-	6600 1400 6550 1400
-Wire Wire Line
-	6600 1300 6550 1300
-Wire Wire Line
-	6550 1200 6600 1200
-Wire Wire Line
-	6600 1100 6550 1100
-Wire Wire Line
-	6550 1000 6600 1000
-Text GLabel 7800 1025 0    60   Input ~ 0
+	6700 2400 6750 2400
+Wire Wire Line
+	6750 2300 6700 2300
+Wire Wire Line
+	6700 2200 6750 2200
+Wire Wire Line
+	6750 2100 6700 2100
+Wire Wire Line
+	6700 2000 6750 2000
+Wire Wire Line
+	6700 1900 6750 1900
+Wire Wire Line
+	6750 1800 6700 1800
+Wire Wire Line
+	6700 1700 6750 1700
+Wire Wire Line
+	6750 1600 6700 1600
+Wire Wire Line
+	6700 1500 6750 1500
+Wire Wire Line
+	6750 1400 6700 1400
+Wire Wire Line
+	6750 1300 6700 1300
+Wire Wire Line
+	6700 1200 6750 1200
+Wire Wire Line
+	6750 1100 6700 1100
+Wire Wire Line
+	6700 1000 6750 1000
+Text GLabel 8025 1025 0    60   Input ~ 0
 PWR_GND
-Text GLabel 7800 1125 0    60   Input ~ 0
+Text GLabel 8025 1125 0    60   Input ~ 0
 PWR_GND
-Text GLabel 7800 1225 0    60   Input ~ 0
+Text GLabel 8025 1225 0    60   Input ~ 0
 PB2/I2C_SCL
-Text GLabel 7800 1325 0    60   Input ~ 0
+Text GLabel 8025 1325 0    60   Input ~ 0
 PB3/I2C_SDA
-Text GLabel 7800 1425 0    60   Input ~ 0
+Text GLabel 8025 1425 0    60   Input ~ 0
 PD6
-Text GLabel 7800 1525 0    60   Input ~ 0
+Text GLabel 8025 1525 0    60   Input ~ 0
 RESET
-Text GLabel 7800 1625 0    60   Input ~ 0
+Text GLabel 8025 1625 0    60   Input ~ 0
 HIB
-Text GLabel 7800 2125 0    60   Input ~ 0
+Text GLabel 8025 2125 0    60   Input ~ 0
 PD0/SSI1CLK
-Text GLabel 7800 2225 0    60   Input ~ 0
+Text GLabel 8025 2225 0    60   Input ~ 0
 PD1/SSI1Fss
-Text GLabel 7800 2325 0    60   Input ~ 0
+Text GLabel 8025 2325 0    60   Input ~ 0
 PD2/SSI1Rx
-Text GLabel 7800 2425 0    60   Input ~ 0
+Text GLabel 8025 2425 0    60   Input ~ 0
 PD3/SSI1Tx
-Text GLabel 7800 1725 0    60   Input ~ 0
+Text GLabel 8025 1725 0    60   Input ~ 0
 PB5
-Text GLabel 7800 1825 0    60   Input ~ 0
+Text GLabel 8025 1825 0    60   Input ~ 0
 PB4
-Text GLabel 7800 1925 0    60   Input ~ 0
+Text GLabel 8025 1925 0    60   Input ~ 0
 PE4
-Text GLabel 7800 2025 0    60   Input ~ 0
+Text GLabel 8025 2025 0    60   Input ~ 0
 PE5
-Text GLabel 7800 2525 0    60   Input ~ 0
+Text GLabel 8025 2525 0    60   Input ~ 0
 PWR_VDD
 Wire Wire Line
-	7800 2525 7850 2525
-Wire Wire Line
-	7850 2425 7800 2425
-Wire Wire Line
-	7800 2325 7850 2325
-Wire Wire Line
-	7850 2225 7800 2225
-Wire Wire Line
-	7800 2125 7850 2125
-Wire Wire Line
-	7850 2025 7800 2025
-Wire Wire Line
-	7800 1925 7850 1925
-Wire Wire Line
-	7800 1825 7850 1825
-Wire Wire Line
-	7850 1725 7800 1725
-Wire Wire Line
-	7800 1625 7850 1625
-Wire Wire Line
-	7850 1525 7800 1525
-Wire Wire Line
-	7800 1425 7850 1425
-Wire Wire Line
-	7850 1325 7800 1325
-Wire Wire Line
-	7800 1225 7850 1225
-Wire Wire Line
-	7850 1125 7800 1125
-Wire Wire Line
-	7800 1025 7850 1025
-Text GLabel 6550 2200 0    60   Input ~ 0
+	8025 2525 8075 2525
+Wire Wire Line
+	8075 2425 8025 2425
+Wire Wire Line
+	8025 2325 8075 2325
+Wire Wire Line
+	8075 2225 8025 2225
+Wire Wire Line
+	8025 2125 8075 2125
+Wire Wire Line
+	8075 2025 8025 2025
+Wire Wire Line
+	8025 1925 8075 1925
+Wire Wire Line
+	8025 1825 8075 1825
+Wire Wire Line
+	8075 1725 8025 1725
+Wire Wire Line
+	8025 1625 8075 1625
+Wire Wire Line
+	8075 1525 8025 1525
+Wire Wire Line
+	8025 1425 8075 1425
+Wire Wire Line
+	8075 1325 8025 1325
+Wire Wire Line
+	8025 1225 8075 1225
+Wire Wire Line
+	8075 1125 8025 1125
+Wire Wire Line
+	8025 1025 8075 1025
+Text GLabel 6700 2200 0    60   Input ~ 0
 PC7
+Wire Notes Line
+	7200 500  7200 3050
+Wire Notes Line
+	7250 3050 8500 3050
+Wire Notes Line
+	7250 3050 7250 500
+Wire Notes Line
+	7250 500  8500 500
 $EndSCHEMATC
